File: I2SHat/I2SHat.kicad_pcb (KiCad board)
At the start: 4 copper layers, 65 x 56 mm, 98 parts, among them J1 TORX142L, J2 TOTX142L, J3 TX_RCA, J4 Raspberry_Pi_2_3, J5 RX_RCA, Q1 BSS138, Q2 BSS138, Q3 BSS138, Q4 BSS138, Q5 BSS138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

Commit message: WIP changes
Other:
- net class Default removed
